File: V2/KiCad_project/OvervoltageProtection.kicad_sch (KiCad schematic)
At the start: 15 parts, among them U501 LM393DR2G

Commit message: Fix rotation for JLCPCB
Add `FT Rotation Offset` fields to components that have a wrong
rotation when ordering from JLCPCB.
Parts:
- D501: FT Rotation Offset (none) -> 180
Changed lines of the file:
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@@
+			)
+		)
+		(property "FT Rotation Offset" "180"
+			(at 81.28 91.44 90)
+			(effects
+				(font
+					(size 1.27 1.27)
+				)
+				(hide yes)
 			)
 		)
